File: PCB/MCU/MCU.kicad_sch (KiCad schematic)
At the start: 0 parts

Commit message: Most of MCU schematic done
Parts:
- added C1, C2: 30p, symbol Device:C
- added C10, C11, C12, C13, C5, C6, C7, C8, C9: 100n, symbol Device:C
- added C14, C15: 10u, symbol Device:C
- added C3, C4: 1u, symbol Device:C
- added J: From Breakout, symbol Connector_Generic:Conn_01x04
- added J1, J10, J2, J3, J4, J5, J6, J7, J8, J9: BTN, symbol Connector_Generic:Conn_01x04
- added J11, J12: ENC, symbol Connector_Generic:Conn_01x04
- added Q1, Q10, Q2, Q3, Q4, Q5, Q6, Q7, Q8, Q9: NTE4153NT1G, Library:SC89-3_0P95X1P7_ONS, symbol Transistor_FET:BSS123
- added R1, R2: 27.4, symbol Device:R
- added R3: 1k, symbol Device:R
- added U1: RP2040, Package_DFN_QFN:QFN-56-1EP_7x7mm_P0.4mm_EP3.2x3.2mm, symbol MCU_RaspberryPi:RP2040
- added U2: W25Q128JVS, Package_SO:SOIC-8_5.3x5.3mm_P1.27mm, symbol Memory_Flash:W25Q128JVS
- added U3: AMS1117-3.3, Package_TO_SOT_SMD:SOT-223-3_TabPin2, symbol Regulator_Linear:AMS1117-3.3
- added Y1: ABLS-12.000MHZ-B4-T, ABLS-12.000MHZ-B4-T:XTAL_ABLS-12.000MHZ-B4-T, symbol Library:ABLS-12.000MHZ-B4-T
Connections:
- new net: J9.2 (Pin_2), Q9.3 (D)
- new net: J10.2 (Pin_2), Q10.3 (D)
- new net: C1.2, U1.20 (XIN), Y1.1
- new net: J1.2 (Pin_2), Q1.3 (D)
- new net: J5.2 (Pin_2), Q5.3 (D)
- new net: C2.2, R3.1, Y1.2
- new net: R3.2, U1.21 (XOUT)
- new net: R2.2, U1.47 (USB_DP)
- new net: J4.2 (Pin_2), Q4.3 (D)
- new net: R1.2, U1.46 (USB_DM)
- new net: J7.2 (Pin_2), Q7.3 (D)
- new net: J3.2 (Pin_2), Q3.3 (D)
- new net: J2.2 (Pin_2), Q2.3 (D)
- new net: J8.2 (Pin_2), Q8.3 (D)
- new net: J6.2 (Pin_2), Q6.3 (D)
- new net +1.1V: C4.1, C5.1, C6.1, U1.23 (DVDD), U1.45 (VREG_VOUT), U1.50 (DVDD)
- new net +3.3V: C10.1, C11.1, C12.1, C13.1, C15.1, C3.1, C7.1, C8.1, C9.1, U1.1 (IOVDD), U1.10 (IOVDD), U1.22 (IOVDD), U1.33 (IOVDD), U1.42 (IOVDD), U1.43 (ADC_AVDD), U1.44 (VREG_VIN), U1.48 (USB_VDD), U1.49 (IOVDD), U2.8 (VCC), U3.2 (VO)
- new net BLED1: Q1.1 (G)
- new net BLED10: Q10.1 (G)
- new net BLED2: Q2.1 (G)
- new net BLED3: Q3.1 (G)
- new net BLED4: Q4.1 (G)
- new net BLED5: Q5.1 (G)
- new net BLED6: Q6.1 (G)
- new net BLED7: Q7.1 (G)
- new net BLED8: Q8.1 (G)
- new net BLED9: Q9.1 (G)
- new net BTN1: J1.3 (Pin_3)
- new net BTN10: J10.3 (Pin_3)
- new net BTN2: J2.3 (Pin_3)
- new net BTN3: J3.3 (Pin_3)
- new net BTN4: J4.3 (Pin_3)
- new net BTN5: J5.3 (Pin_3)
- new net BTN6: J6.3 (Pin_3)
- new net BTN7: J7.3 (Pin_3)
- new net BTN8: J8.3 (Pin_3)
- new net BTN9: J9.3 (Pin_3)
- new net D+: J.2 (Pin_2), R2.1
- new net D-: J.3 (Pin_3), R1.1
- new net GND: C1.1, C10.2, C11.2, C12.2, C13.2, C14.2, C15.2, C2.1, C3.2, C4.2, C5.2, C6.2, C7.2, C8.2, C9.2, J.4 (Pin_4), J1.4 (Pin_4), J10.4 (Pin_4), J11.4 (Pin_4), J12.4 (Pin_4), J2.4 (Pin_4), J3.4 (Pin_4), J4.4 (Pin_4), J5.4 (Pin_4), J6.4 (Pin_4), J7.4 (Pin_4), J8.4 (Pin_4), J9.4 (Pin_4), Q1.2 (S), Q10.2 (S), Q2.2 (S), Q3.2 (S), Q4.2 (S), Q5.2 (S), Q6.2 (S), Q7.2 (S), Q8.2 (S), Q9.2 (S), U1.19 (TESTEN), U1.57 (GND), U2.4 (GND), U3.1 (GND)
- new net QE1A: J11.2 (Pin_2), U1.38 (GPIO26/ADC0)
- new net QE1B: J11.3 (Pin_3), U1.39 (GPIO27/ADC1)
- new net QE2A: J12.2 (Pin_2), U1.40 (GPIO28/ADC2)
- new net QE2B: J12.3 (Pin_3), U1.41 (GPIO29/ADC3)
- new net QSPI_SCLK: U1.52 (QSPI_SCLK), U2.6 (CLK)
- new net QSPI_SD0: U1.53 (QSPI_SD0), U2.5 (DI/IO_{0})
- new net QSPI_SD1: U1.55 (QSPI_SD1), U2.2 (DO/IO_{1})
- new net QSPI_SD2: U1.54 (QSPI_SD2), U2.3 (~{WP}/IO_{2})
- new net QSPI_SD3: U1.51 (QSPI_SD3), U2.7 (~{HOLD}/~{RESET}/IO_{3})
- new net QSPI_SS: U1.56 (~{QSPI_SS}), U2.1 (~{CS})
- new net VBUS: C14.1, J.1 (Pin_1), J1.1 (Pin_1), J10.1 (Pin_1), J11.1 (Pin_1), J12.1 (Pin_1), J2.1 (Pin_1), J3.1 (Pin_1), J4.1 (Pin_1), J5.1 (Pin_1), J6.1 (Pin_1), J7.1 (Pin_1), J8.1 (Pin_1), J9.1 (Pin_1), U3.3 (VI)

Commit message: Final Schematic Touches
Parts:
- added J14: IO Access, symbol Connector_Generic:Conn_02x06_Top_Bottom
- renumbered J to J13
Connections:
- net +1.1V: now also U1.26 (RUN)
- net BLED1: now also U1.3 (GPIO1)
- net BLED10: now also U1.30 (GPIO19)
- net BLED2: now also U1.5 (GPIO3)
- net BLED3: now also U1.7 (GPIO5)
- net BLED4: now also U1.9 (GPIO7)
- net BLED5: now also U1.12 (GPIO9)
- net BLED6: now also U1.14 (GPIO11)
- net BLED7: now also U1.16 (GPIO13)
- net BLED8: now also U1.18 (GPIO15)
- net BLED9: now also U1.28 (GPIO17)
- net BTN1: now also U1.2 (GPIO0)
- net BTN10: now also U1.29 (GPIO18)
- net BTN2: now also U1.4 (GPIO2)
- net BTN3: now also U1.6 (GPIO4)
- net BTN4: now also U1.8 (GPIO6)
- net BTN5: now also U1.11 (GPIO8)
- net BTN6: now also U1.13 (GPIO10)
- net BTN7: now also U1.15 (GPIO12)
- net BTN8: now also U1.17 (GPIO14)
- net BTN9: now also U1.27 (GPIO16)
- net GND: now also J14.10 (Pin_10), J14.11 (Pin_11), J14.12 (Pin_12), J14.7 (Pin_7), J14.8 (Pin_8), J14.9 (Pin_9)
- net at U1.31 (GPIO20): now also J14.1 (Pin_1)
- net at U1.32 (GPIO21): now also J14.2 (Pin_2)
- net at U1.34 (GPIO22): now also J14.3 (Pin_3)
- net at U1.35 (GPIO23): now also J14.4 (Pin_4)
- net at U1.36 (GPIO24): now also J14.5 (Pin_5)
- net at U1.37 (GPIO25): now also J14.6 (Pin_6)
